File: ams-master-pcb.sch (EAGLE design)
At the start: 220 parts, among them J1 M50-3601042, J2 TE-776087, J3 MUSBD11130, Q1 STD45P4LLF6AG, Q2 BSS138, Q3 BSS138, Q4 BSS138, Q7 FQD3P50, Q8 FQD3P50, U1 PDS1-S5-S5-M-TR, U10 ISO7221, U11 ISO7221, U13 MCP2562FD, U14 SN74LVC541A, U16 LM3671MF-3.3/NOPB, U17 SN74LVC1G02DBV, U18 LM3671MF-1.2/NOPB, U2 SN74LVC1G32DBV, U22 FAN3214, U23 FAN3214, U24 CSD17506Q5A, U25 CSD17506Q5A, U27 CSD17506Q5A, U3 SN74LVC1G08DBV, U30 ISO7221, U31 ISO7221, U32 PDS1-S5-S5-M-TR, U33 ISO7221, U34 ISO7221, U35 PDS1-S5-S5-M-TR, U36 ADC121S021, U37 ADC121S021, U38 FT232RL, U42 TPS54540DDARQ1, U5 CD4050BD, U6 CD4050BD, U7 MCP2562FD, U8 ADUM3160BRWZ-RL, U9 CD4050BD, Y2 16MHz

Commit message: Push to work on laptop
Parts:
- removed U9: CD4050BD, FormE:CD4050BD
- added C24, C25, C26, C27: 0.1uF, rcl:C-USC0603K
Connections:
- removed net VCC: C96.1, C97.1, R52.2, U42.VIN
- new net N$34: U4IO.CAN2TX
- net +15V: now also C24.1, C25.1, C26.1, C96.1, C97.1, R52.2, U22G$3.VCC, U23G$3.VCC, U42.VIN, U6POWER.VCC
- net +3V3: now also C27.1, U5POWER.VCC
- net GND: now also C24.2, C25.2, C26.2, C27.2, U22G$3.GND, U23G$3.GND, U5POWER.GND, U6POWER.GND
- net INDICATOR_3: now also U4IO.N2HET1[12]/MII_CRS/RMII_CRS_DV
- net N$11: now also U5A.IN; no longer U9D.IN
- net SC_FROM_OUTSIDE_SENSE: now also U5A.OUT; no longer U9D.OUT
Other:
- note added: "Look at 100V rated MOSFETS?"
- moved on the sheet: C21, C22, C23

Commit message: Output buffers
Parts:
- added D6, D8: BAV21W, FormE:BAV21W
- added Q5, Q6: BSS138, FormE:BSS138
- added R11, R23, R24, R4: 10k, rcl:R-US_R0603
- added R16, R25: DNP/10k, rcl:R-US_R0603
Connections:
- removed net 5KW: J2.P1
- new net 5KW_3V3: Q5.S, R11.2
- new net 5KW_GLV: D6.CATHODE, J2.P1, R16.2
- new net CURRENT_SHORT_3V3: Q6.S, R24.2
- new net CURRENT_SHORT_GLV: D8.CATHODE, J2.P9, R25.2
- new net N$35: Q5.D, R4.2, U6B.IN
- new net N$36: D6.ANODE, U6B.OUT
- new net N$37: Q6.D, R23.2, U6A.IN
- new net N$38: D8.ANODE, U6A.OUT
- net +15V: now also R23.1, R4.1
- net +3V3: now also Q5.G, Q6.G, R11.1, R24.1
- net GND: now also R16.1, R25.1
Other:
- moved on the sheet: U6A, U6B

Commit message: Nearly done
Parts:
- added H3: 502443-0870, FormE:MOLEX_502443-0870
- added LED14, LED15, LED16: GREEN, FormE:LEDCHIP-LED0805
- added R26, R27, R28: 1k, rcl:R-US_R0603
- added R29, R33: 150k, rcl:R-US_R0805
- LED1: value RED -> BLUE
Connections:
- removed net N$29: U4IO.CAN2RX
- removed net N$34: U4IO.CAN2TX
- new net N$42: LED14.C, R26.2
- new net N$43: LED15.C, R27.2
- new net N$44: LED16.C, R28.2
- new net N$45: R29.2, R98.1
- new net N$48: R103.1, R33.2
- net +15V: now also H3.1
- net +3V3: now also H3.3; no longer R11.1, R24.1
- net +5V: now also H3.2
- net +5V/1: now also LED16.A
- net +5V/2: now also LED15.A
- net +5V/3: now also LED14.A
- net 5KW_3V3: now also H3.6, R11.1, U4IO.GIOB[1]/USB1.PORTPOWER; no longer R11.2
- net CURRENT_SENSE_-750_TO_750A: now also H3.5
- net CURRENT_SENSE_-75_TO_75A: now also H3.4
- net CURRENT_SHORT_3V3: now also H3.7, R24.1, U4IO.GIOB[2]; no longer R24.2
- net GND: now also H3.8, R11.2, R24.2
- net GND1: now also R28.1
- net GND2: now also R27.1
- net GND3: now also R26.1
- net N$101: no longer SV1.3
- net N$102: now also SV1.3
- net N$111: now also SV2.3
- net N$112: no longer SV2.3
- net N$114: now also R33.1; no longer R103.1
- net N$117: now also R29.1; no longer R98.1
Other:
- note added: "Current Sensor"
- note added: "LOOK AT HOW OLD AMS DID VOLTAGE SESING (2 SPI OR 1)"
- note added: "Look at 100V rated MOSFETS? https://www.gigavac.com/sites/default/files/catalog/spec_sheet/gx14.pdf Looks like it can have 55V Back EMF even with Suppression."
- note added: "SOURCE 400v Connectors"
- note added: "Still need to pin out BMS communication"
- note removed: "ADD LEDs SOURCE 400v components"
- note removed: "Look at 100V rated MOSFETS?"
- moved on the sheet: C21, C22, C23, C27, C64, C65, D11, D13, JP12, R11, R24, R57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

Commit message: Schematic done, will begin routing
Parts:
- added JP6, JP7: 0R, FormE:TWO-WAY-JUMPER-0603
Connections:
- removed net BATTERY_VOLTAGE_MISO: U33.OUTB
- removed net OPT_BATTERY_VOLTAGE_MONITOR_CS: U4IO.N2HET1[3]/SPI4NCS[0]/USB2.SPEED/USB_FUNC.PUENON/N2HET2[10]/EQEP2B
- removed net OPT_BATTERY_VOLTAGE_MONITOR_MISO: U4IO.N2HET1[5]/SPI4SOMI[0]/N2HET2[12]/EPWM3B
- removed net OPT_BATTERY_VOLTAGE_MONITOR_SCK: U4IO.N2HET1[0]/SPI4CLK/EPWM2B
- removed net VOLTAGE_MONITOR_MISO: U4IO.MIBSPI1SOMI[0]
- removed net VOLTAGE_MONITOR_SCLK: U4IO.MIBSPI1CLK
- new net BATTERY_VOLTAGE_MONITOR_MISO: U33.OUTB, U4IO.N2HET1[5]/SPI4SOMI[0]/N2HET2[12]/EPWM3B
- new net BMS_UART_RX: JP7.P$1, U4IO.N2HET1[6]/SCIRX/EPWM5A
- new net BMS_UART_TX: JP6.P$1, U4IO.N2HET1[13]/SCITX/EPWM5B
- net BATTERY_VOLTAGE_MONITOR_CS: now also U4IO.N2HET1[3]/SPI4NCS[0]/USB2.SPEED/USB_FUNC.PUENON/N2HET2[10]/EQEP2B
- net BATTERY_VOLTAGE_MONITOR_SCLK: now also U4IO.N2HET1[0]/SPI4CLK/EPWM2B
- net BMS_CAN_RX: now also JP7.P$3, U4IO.CAN2RX
- net BMS_CAN_TX: now also JP6.P$3, U4IO.CAN2TX
- net BMS_RX: now also JP7.P$2
- net BMS_TX: now also JP6.P$2
- net VEHICLE_VOLTAGE_MISO: now also U4IO.MIBSPI1SOMI[0]
- net VEHICLE_VOLTAGE_MONITOR_SCLK: now also U4IO.MIBSPI1CLK
- net WAKEUP: now also U4IO.GIOB[3]/USB2.RCV/USB_FUNC.RXDI
Other:
- note added: "@400V outputs 5.263V"
- note added: "Connection after the fuse to offer protection to the IMD"
- note removed: "Still need to pin out BMS communication"

Commit message: Added some comments
Other:
- note added: "LOOK AT HOW OLD AMS DID VOLTAGE SESING (2 SPI OR 1) Looks like they implemented both muxd into the 1 channel, 2 might be easier to code? @Hutch"
- note removed: "LOOK AT HOW OLD AMS DID VOLTAGE SESING (2 SPI OR 1)"
Changed lines of the file:
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@@
 <wire x1="378.46" y1="-279.4" x2="378.46" y2="-205.74" width="2.54" layer="97"/>
 <wire x1="162.56" y1="-170.18" x2="378.46" y2="-170.18" width="2.54" layer="97"/>
-<text x="-759.46" y="104.14" size="2.54" layer="94">LOOK AT HOW OLD AMS DID VOLTAGE SESING (2 SPI OR 1)</text>
-<text x="264.16" y="193.04" size="2.54" layer="94">LOOK AT HOW OLD AMS DID VOLTAGE SESING (2 SPI OR 1)</text>
+<text x="-779.78" y="91.44" size="2.54" layer="94">LOOK AT HOW OLD AMS DID VOLTAGE SESING (2 SPI OR 1)
+Looks like they implemented both muxd into the 1 channel, 2 might be easier to code?
+@Hutch</text>
 <wire x1="121.92" y1="449.58" x2="378.46" y2="449.58" width="2.54" layer="97"/>
 <wire x1="378.46" y1="449.58" x2="378.46" y2="297.18" width="2.54" layer="97"/>

Commit message: Started Routing
Connections:
- net N$1 renamed NEG_GATE
- net N$20 renamed PRE_FET
- net N$4 renamed NEG_FET
- net N$5 renamed POS_FET
- net N$6 renamed POS_GATE
Changed lines of the file:
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@@
 </segment>
 </net>
-<net name="N$4" class="0">
+<net name="NEG_FET" class="0">
 <segment>
 <pinref part="U25" gate="A" pin="D"/>
@@
 </segment>
 </net>
-<net name="N$20" class="0">
+<net name="PRE_FET" class="0">
 <segment>
 <pinref part="U27" gate="A" pin="D"/>
@@
 </segment>
 </net>
-<net name="N$1" class="0">
+<net name="NEG_GATE" class="0">
 <segment>
 <pinref part="U22" gate="B" pin="OUT"/>
@@
 </segment>
 </net>
-<net name="N$5" class="0">
+<net name="POS_FET" class="0">
 <segment>
 <pinref part="H6" gate="G$1" pin="2"/>
@@
 </segment>
 </net>
-<net name="N$6" class="0">
+<net name="POS_GATE" class="0">
 <segment>
 <pinref part="U24" gate="A" pin="G"/>

Commit message: Added some comments to the schematic, good talking points
Other:
- note added: "Current Short Indicator??"
- note added: "If we want to buffer the input from the current sensor board we could use these?"
- note added: "low-side mosfet controller, don't really have a good use for it, unless we want to power the fans?"
Changed lines of the file:
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@@
 <text x="-403.86" y="73.66" size="1.778" layer="97">Connection after the fuse to offer
 protection to the IMD</text>
+<text x="-60.96" y="-78.74" size="1.778" layer="91">Current Short Indicator??</text>
+<text x="170.18" y="368.3" size="1.778" layer="91">If we want to buffer the input from the current sensor board we could use these?</text>
+<text x="538.48" y="-15.24" size="1.778" layer="91">low-side mosfet controller, don't really have a good use for it,
+unless we want to power the fans?</text>
 </plain>
 <instances>

Commit message: ez
Parts:
- removed JP5: (no value), adafruit:PINHD-1X6CB
- removed SV1, SV2: (no value), con-lstb:MA04-1
- added J4, J6: MOLEX_43650-0416MOLEX_43650-0416_0_0, FormE:MOLEX_43650-0416MOLEX_43650-0416_0_0
- added J7: 43650-0616, FormE:MOLEX_43650-0616
Connections:
- removed net BATTERY_VOLTAGE_MONITOR_MISO: U33.OUTB, U4IO.N2HET1[5]/SPI4SOMI[0]/N2HET2[12]/EPWM3B
- removed net BATTERY_VOLTAGE_MONITOR_SCLK: U34.INA, U4IO.N2HET1[0]/SPI4CLK/EPWM2B
- removed net VEHICLE_VOLTAGE_MISO: U30.OUTB, U4IO.MIBSPI1SOMI[0]
- removed net VEHICLE_VOLTAGE_MONITOR_SCLK: U31.INA, U4IO.MIBSPI1CLK
- new net VOLTAGE_MONITOR_MISO: U30.OUTB, U33.OUTB, U4IO.MIBSPI1SOMI[0]
- new net VOLTAGE_MONITOR_SCLK: U31.INA, U34.INA, U4IO.MIBSPI1CLK
- net +5V/1: now also J7.4; no longer JP5.4
- net BATTERY_VOLTAGE_MONITOR_CS: no longer U4IO.N2HET1[3]/SPI4NCS[0]/USB2.SPEED/USB_FUNC.PUENON/N2HET2[10]/EQEP2B
- net BMS_FAULT_HV: now also J7.5; no longer JP5.5
- net BMS_RX_HV: now also J7.2; no longer JP5.2
- net BMS_TX_HV: now also J7.3; no longer JP5.3
- net GND1: now also J7.6; no longer JP5.6
- net GND2: now also J4.3, J4.4; no longer SV1.1, SV1.2
- net GND3: now also J6.3, J6.4; no longer SV2.1, SV2.2
- net N$102: now also J4.1, J4.2; no longer SV1.3, SV1.4
- net N$111: now also J6.2; no longer SV2.3
- net N$112: now also J6.1; no longer SV2.4
- net WAKEUP_HV: now also J7.1; no longer JP5.1
Other:
- note removed: "LOOK AT HOW OLD AMS DID VOLTAGE SESING (2 SPI OR 1) Looks like they implemented both muxd into the 1 channel, 2 might be easier to code? @Hutch"
