File: ams-master-pcb.sch (EAGLE design)
At the start: 244 parts, among them J1 M50-3601042, J2 TE-776087, J3 MUSBD11130, J4 MOLEX_43650-0416MOLEX_43650-0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, J6 MOLEX_43650-0416MOLEX_43650-0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, J7 43650-0616, Q1 STD45P4LLF6AG, Q2 BSS138, Q3 BSS138, Q4 BSS138, Q5 BSS138, Q6 BSS138, Q7 FQD3P50, Q8 FQD3P50, U1 PDS1-S5-S5-M-TR, U10 ISO7221, U11 ISO7221, U13 MCP2562FD, U14 SN74LVC541A, U16 LM3671MF-3.3/NOPB, U17 SN74LVC1G02DBV, U18 LM3671MF-1.2/NOPB, U2 SN74LVC1G32DBV, U22 FAN3214, U23 FAN3214, U24 CSD17506Q5A, U25 CSD17506Q5A, U27 CSD17506Q5A, U3 SN74LVC1G08DBV, U30 ISO7221, U31 ISO7221, U32 PDS1-S5-S5-M-TR, U33 ISO7221, U34 ISO7221, U35 PDS1-S5-S5-M-TR, U36 ADC121S021, U37 ADC121S021, U38 FT232RL, U42 TPS54540DDARQ1, U5 CD4050BD, U6 CD4050BD, U7 MCP2562FD, U8 ADUM3160BRWZ-RL, Y2 16MHz

Commit message: rough
Parts:
- added C28: 4.7uF, rcl:C-USC0603K
Connections:
- net BMS_CAN_N renamed HV_BMS_CAN_N
- net BMS_CAN_P renamed HV_BMS_CAN_P
- new net HV_BMS_CAN_RX: JP1.P$3, U13.RXD
- new net HV_BMS_CAN_TX: JP2.P$3, U13.TXD
- net +5V/1: now also C28.1
- net BMS_CAN_RX: no longer JP1.P$3, U13.RXD
- net BMS_CAN_TX: no longer JP2.P$3, U13.TXD
- net BMS_FAULT: now also U11.OUTB; no longer U10.OUTB
- net BMS_FAULT_HV: now also U11.INB; no longer U10.INB
- net BMS_RX: now also U10.OUTB; no longer U11.OUTB
- net GND1: now also C28.2
- net N$31: now also U10.INB; no longer U11.INB
Other:
- moved on the sheet: JP7

Commit message: routing
Parts:
- removed S3: TE-FSM4JSMATR, FormE:TE-FSM4JSMATR
- added S2: 147873-2, FormE:TE-147873-2
Connections:
- net GND: now also S2.2; no longer S3.3, S3.4
- net N$63: now also S2.1; no longer S3.1, S3.2
Changed lines of the file:
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@@
 <attribute name="PARTNO" value="ERJ-3EKF2201V"/>
 </part>
-<part name="S3" library="FormE" deviceset="TE-FSM4JSMATR" device="">
-<attribute name="PARTNO" value="FSM4JSMATR"/>
-</part>
 <part name="LED4" library="FormE" deviceset="LED" device="CHIP-LED0805" value="RED">
 <attribute name="PARTNO" value="5988110107F"/>
@@
 <attribute name="PARTNO" value="GRM188R61A475KE15D"/>
 </part>
+<part name="S2" library="FormE" deviceset="TE-147873-2" device="" value="147873-2">
+<attribute name="PARTNO" value="147873-2"/>
+</part>
 </parts>
 <sheets>
@@
 <attribute name="VALUE" x="132.842" y="280.67" size="1.778" layer="96" rot="MR270"/>
 </instance>
-<instance part="S3" gate="G$1" x="152.4" y="269.24" smashed="yes" rot="MR0">
-<attribute name="PARTNO" x="152.4" y="269.24" size="1.778" layer="96" rot="MR0" display="off"/>
-<attribute name="NAME" x="154.94" y="274.32" size="1.778" layer="95" rot="MR0"/>
-</instance>
 <instance part="LED4" gate="G$1" x="149.86" y="251.46" smashed="yes" rot="R270">
 <attribute name="PARTNO" x="149.86" y="251.46" size="1.778" layer="96" rot="R180" display="off"/>
@@
 <attribute name="VALUE" x="-580.136" y="295.529" size="1.778" layer="96" rot="MR0"/>
 </instance>
+<instance part="S2" gate="G$1" x="152.4" y="269.24" smashed="yes">
+<attribute name="PARTNO" x="152.4" y="269.24" size="1.778" layer="96" display="off"/>
+<attribute name="NAME" x="152.4" y="271.78" size="1.778" layer="95" align="bottom-center"/>
+<attribute name="VALUE" x="152.4" y="265.938" size="1.778" layer="96" align="bottom-center"/>
+</instance>
 </instances>
 <busses>
@@
 <segment>
 <pinref part="GND18" gate="1" pin="GND"/>
-<wire x1="160.02" y1="261.62" x2="160.02" y2="266.7" width="0.1524" layer="91"/>
-<wire x1="160.02" y1="266.7" x2="157.48" y2="266.7" width="0.1524" layer="91"/>
+<wire x1="160.02" y1="261.62" x2="160.02" y2="269.24" width="0.1524" layer="91"/>
 <wire x1="157.48" y1="269.24" x2="160.02" y2="269.24" width="0.1524" layer="91"/>
-<wire x1="160.02" y1="269.24" x2="160.02" y2="266.7" width="0.1524" layer="91"/>
-<junction x="160.02" y="266.7"/>
-<pinref part="S3" gate="G$1" pin="4"/>
-<pinref part="S3" gate="G$1" pin="3"/>
+<pinref part="S2" gate="G$1" pin="2"/>
 </segment>
 <segment>
@@
 <net name="N$63" class="0">
 <segment>
-<wire x1="147.32" y1="266.7" x2="144.78" y2="266.7" width="0.1524" layer="91"/>
-<wire x1="144.78" y1="266.7" x2="144.78" y2="269.24" width="0.1524" layer="91"/>
-<wire x1="144.78" y1="269.24" x2="147.32" y2="269.24" width="0.1524" layer="91"/>
 <pinref part="R31" gate="G$1" pin="2"/>
-<wire x1="142.24" y1="269.24" x2="144.78" y2="269.24" width="0.1524" layer="91"/>
-<junction x="144.78" y="269.24"/>
-<pinref part="S3" gate="G$1" pin="1"/>
-<pinref part="S3" gate="G$1" pin="2"/>
+<wire x1="142.24" y1="269.24" x2="147.32" y2="269.24" width="0.1524" layer="91"/>
+<pinref part="S2" gate="G$1" pin="1"/>
 </segment>
 </net>

Commit message: Continued layout
Connections:
- net 5KW_3V3: now also U14A.IN
- net CURRENT_SENSE_-750_TO_750A: now also H3.4; no longer H3.5
- net CURRENT_SENSE_-75_TO_75A: now also H3.5; no longer H3.4
- net INDICATOR_2: no longer U4IO.N2HET1[30]/MII_RX_DV/USB1.SPEED/EQEP2S
- net INDICATOR_3: no longer U14A.IN
Changed lines of the file:
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@@
 <pinref part="U14" gate="F" pin="IN"/>
-</segment>
-<segment>
-<pinref part="U4" gate="IO" pin="N2HET1[30]/MII_RX_DV/USB1.SPEED/EQEP2S"/>
-<wire x1="251.46" y1="106.68" x2="345.44" y2="106.68" width="0.1524" layer="91"/>
-<label x="345.44" y="106.68" size="1.778" layer="95" rot="MR0"/>
 </segment>
 </net>
@@
 </net>
 <net name="INDICATOR_3" class="0">
-<segment>
-<pinref part="U14" gate="A" pin="IN"/>
-<wire x1="-83.82" y1="-81.28" x2="-124.46" y2="-81.28" width="0.1524" layer="91"/>
-<label x="-124.46" y="-81.28" size="1.778" layer="95"/>
-</segment>
 <segment>
 <pinref part="U4" gate="IO" pin="N2HET1[12]/MII_CRS/RMII_CRS_DV"/>
@@
 </segment>
 <segment>
-<pinref part="H3" gate="G$1" pin="4"/>
-<wire x1="144.78" y1="406.4" x2="193.04" y2="406.4" width="0.1524" layer="91"/>
-<label x="193.04" y="406.4" size="1.778" layer="95" rot="MR0"/>
+<wire x1="144.78" y1="403.86" x2="193.04" y2="403.86" width="0.1524" layer="91"/>
+<pinref part="H3" gate="G$1" pin="5"/>
+<label x="193.04" y="403.86" size="1.778" layer="95"/>
 </segment>
 </net>
@@
 </segment>
 <segment>
-<pinref part="H3" gate="G$1" pin="5"/>
-<wire x1="144.78" y1="403.86" x2="193.04" y2="403.86" width="0.1524" layer="91"/>
-<label x="193.04" y="403.86" size="1.778" layer="95" rot="MR0"/>
+<wire x1="144.78" y1="406.4" x2="193.04" y2="406.4" width="0.1524" layer="91"/>
+<pinref part="H3" gate="G$1" pin="4"/>
+<label x="193.04" y="406.4" size="1.778" layer="95" rot="MR0"/>
 </segment>
 </net>
@@
 <label x="40.64" y="63.5" size="1.778" layer="95"/>
 </segment>
-</net>
+<segment>
+<pinref part="U14" gate="A" pin="IN"/>
+<wire x1="-83.82" y1="-81.28" x2="-114.3" y2="-81.28" width="0.1524" layer="91"/>
+<label x="-114.3" y="-81.28" size="1.778" layer="95"/>
+</segment>
+</net>

Commit message: CAM processed
Parts:
- removed H3: 502443-0870, FormE:MOLEX_502443-0870
- added JP5: (no value), pinhead:PINHD-1X8/90
Connections:
- removed net INDICATOR_3: U4IO.N2HET1[12]/MII_CRS/RMII_CRS_DV
- net +15V: now also JP5.8; no longer H3.1
- net +3V3: now also JP5.6; no longer H3.3
- net +5V: now also JP5.7; no longer H3.2
- net 5KW_3V3: now also JP5.3; no longer H3.6
- net CURRENT_SENSE_-750_TO_750A: now also JP5.5; no longer H3.4
- net CURRENT_SENSE_-75_TO_75A: now also JP5.4; no longer H3.5
- net CURRENT_SHORT_3V3: now also JP5.2; no longer H3.7
- net GND: now also JP5.1; no longer H3.8
- net INDICATOR_2: now also U4IO.N2HET1[12]/MII_CRS/RMII_CRS_DV
Other:
- moved on the sheet: U5D, U5E
Changed lines of the file:
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@@
 <part name="GND47" library="supply1" deviceset="GND" device=""/>
 <part name="GND49" library="supply1" deviceset="GND" device=""/>
-<part name="H3" library="FormE" deviceset="MOLEX_502443-0870" device="" value="502443-0870">
-<attribute name="PARTNO" value="5024430870"/>
-</part>
 <part name="GND50" library="supply1" deviceset="GND" device=""/>
 <part name="+3V20" library="supply1" deviceset="+3V3" device=""/>
@@
 <attribute name="PARTNO" value="147873-2"/>
 </part>
+<part name="JP5" library="pinhead" library_urn="urn:adsk.eagle:library:325" deviceset="PINHD-1X8" device="/90" package3d_urn="urn:adsk.eagle:package:22413/2"/>
 </parts>
 <sheets>
@@
 <attribute name="NAME" x="234.95" y="-240.03" size="1.778" layer="95" font="vector" rot="R180" align="bottom-center"/>
 </instance>
-<instance part="U5" gate="D" x="160.02" y="342.9" smashed="yes" rot="MR0">
-<attribute name="NAME" x="158.75" y="351.79" size="1.778" layer="95" font="vector" rot="MR0" align="bottom-center"/>
+<instance part="U5" gate="D" x="154.94" y="353.06" smashed="yes" rot="MR180">
+<attribute name="NAME" x="156.21" y="344.17" size="1.778" layer="95" font="vector" rot="MR180" align="bottom-center"/>
 </instance>
-<instance part="U5" gate="E" x="160.02" y="325.12" smashed="yes" rot="MR0">
-<attribute name="NAME" x="158.75" y="334.01" size="1.778" layer="95" font="vector" rot="MR0" align="bottom-center"/>
+<instance part="U5" gate="E" x="154.94" y="337.82" smashed="yes" rot="MR180">
+<attribute name="NAME" x="156.21" y="328.93" size="1.778" layer="95" font="vector" rot="MR180" align="bottom-center"/>
 </instance>
 <instance part="U5" gate="F" x="154.94" y="358.14" smashed="yes">
@@
 <attribute name="VALUE" x="121.92" y="-274.32" size="1.778" layer="96" rot="MR0"/>
 </instance>
-<instance part="H3" gate="G$1" x="144.78" y="406.4" smashed="yes" rot="MR0">
-<attribute name="PARTNO" x="144.78" y="406.4" size="1.778" layer="96" rot="MR0" display="off"/>
-<attribute name="NAME" x="147.32" y="421.64" size="1.778" layer="95" rot="MR0"/>
-<attribute name="VALUE" x="147.32" y="419.1" size="1.778" layer="96" rot="MR0"/>
-</instance>
 <instance part="GND50" gate="1" x="154.94" y="388.62" smashed="yes">
 <attribute name="VALUE" x="152.4" y="386.08" size="1.778" layer="96"/>
@@
 <attribute name="VALUE" x="152.4" y="265.938" size="1.778" layer="96" align="bottom-center"/>
 </instance>
+<instance part="JP5" gate="A" x="142.24" y="406.4" smashed="yes" rot="R180">
+<attribute name="NAME" x="148.59" y="393.065" size="1.778" layer="95" rot="R180"/>
+<attribute name="VALUE" x="148.59" y="419.1" size="1.778" layer="96" rot="R180"/>
+</instance>
 </instances>
 <busses>
@@
 </segment>
 <segment>
-<pinref part="H3" gate="G$1" pin="8"/>
 <wire x1="144.78" y1="396.24" x2="154.94" y2="396.24" width="0.1524" layer="91"/>
 <wire x1="154.94" y1="396.24" x2="154.94" y2="391.16" width="0.1524" layer="91"/>
 <pinref part="GND50" gate="1" pin="GND"/>
+<pinref part="JP5" gate="A" pin="1"/>
 </segment>
 </net>
@@
 </segment>
 <segment>
-<pinref part="H3" gate="G$1" pin="3"/>
 <wire x1="144.78" y1="408.94" x2="157.48" y2="408.94" width="0.1524" layer="91"/>
 <wire x1="157.48" y1="408.94" x2="157.48" y2="411.48" width="0.1524" layer="91"/>
 <pinref part="+3V20" gate="G$1" pin="+3V3"/>
+<pinref part="JP5" gate="A" pin="6"/>
 </segment>
 </net>
@@
 </segment>
 <segment>
-<pinref part="H3" gate="G$1" pin="1"/>
 <wire x1="144.78" y1="414.02" x2="152.4" y2="414.02" width="0.1524" layer="91"/>
 <wire x1="152.4" y1="414.02" x2="152.4" y2="416.56" width="0.1524" layer="91"/>
 <pinref part="P+18" gate="1" pin="+15V"/>
+<pinref part="JP5" gate="A" pin="8"/>
 </segment>
 </net>
@@
 </segment>
 <segment>
-<pinref part="H3" gate="G$1" pin="2"/>
 <wire x1="144.78" y1="411.48" x2="154.94" y2="411.48" width="0.1524" layer="91"/>
 <wire x1="154.94" y1="411.48" x2="154.94" y2="414.02" width="0.1524" layer="91"/>
 <pinref part="P+17" gate="1" pin="+5V"/>
+<pinref part="JP5" gate="A" pin="7"/>
 </segment>
 </net>
@@
 <pinref part="U14" gate="F" pin="IN"/>
 </segment>
+<segment>
+<pinref part="U4" gate="IO" pin="N2HET1[12]/MII_CRS/RMII_CRS_DV"/>
+<wire x1="251.46" y1="134.62" x2="345.44" y2="134.62" width="0.1524" layer="91"/>
+<label x="345.44" y="134.62" size="1.778" layer="95" rot="MR0"/>
+</segment>
 </net>
 <net name="N$3" class="0">
@@
 </segment>
 </net>
-<net name="INDICATOR_3" class="0">
-<segment>
-<pinref part="U4" gate="IO" pin="N2HET1[12]/MII_CRS/RMII_CRS_DV"/>
-<wire x1="251.46" y1="134.62" x2="345.44" y2="134.62" width="0.1524" layer="91"/>
-<label x="345.44" y="134.62" size="1.778" layer="95" rot="MR0"/>
-</segment>
-</net>
 <net name="N$23" class="0">
 <segment>
@@
 <segment>
 <wire x1="144.78" y1="403.86" x2="193.04" y2="403.86" width="0.1524" layer="91"/>
-<pinref part="H3" gate="G$1" pin="5"/>
 <label x="193.04" y="403.86" size="1.778" layer="95"/>
+<pinref part="JP5" gate="A" pin="4"/>
 </segment>
 </net>
@@
 <segment>
 <wire x1="144.78" y1="406.4" x2="193.04" y2="406.4" width="0.1524" layer="91"/>
-<pinref part="H3" gate="G$1" pin="4"/>
 <label x="193.04" y="406.4" size="1.778" layer="95" rot="MR0"/>
+<pinref part="JP5" gate="A" pin="5"/>
 </segment>
 </net>
@@
 </segment>
 <segment>
-<pinref part="H3" gate="G$1" pin="6"/>
 <wire x1="144.78" y1="401.32" x2="193.04" y2="401.32" width="0.1524" layer="91"/>
 <label x="193.04" y="401.32" size="1.778" layer="95" rot="MR0"/>
+<pinref part="JP5" gate="A" pin="3"/>
 </segment>
 <segment>
@@
 </segment>
 <segment>
-<pinref part="H3" gate="G$1" pin="7"/>
 <wire x1="144.78" y1="398.78" x2="193.04" y2="398.78" width="0.1524" layer="91"/>
 <label x="193.04" y="398.78" size="1.778" layer="95" rot="MR0"/>
+<pinref part="JP5" gate="A" pin="2"/>
 </segment>
 <segment>
@@
 </sheet>
 </sheets>
+<errors>
+</errors>
 </schematic>
 </drawing>
@@
 will not be understood (or retained) with this version.
 </note>
+<note version="8.3" severity="warning">
+Since Version 8.3, EAGLE supports the association of 3D packages
+with devices in libraries, schematics, and board files. Those 3D
+packages will not be understood (or retained) with this version.
+</note>
 </compatibility>
