File: ams-master-pcb.brd (EAGLE design)
At the start: 203.2 x 101.6 mm, 244 parts, among them J1 M50-3601042, J2 TE-776087, J3 MUSBD11130, Q1 STD45P4LLF6AG, Q2 BSS138, Q3 BSS138, Q4 BSS138, Q5 BSS138, Q6 BSS138, Q7 FQD3P50, Q8 FQD3P50, U1 PDS1-S5-S5-M-TR, U10 ISO7221, U11 ISO7221, U13 MCP2562FD, U14 SN74LVC541A, U16 LM3671MF-3.3/NOPB, U17 SN74LVC1G02DBV, U18 LM3671MF-1.2/NOPB, U2 SN74LVC1G32DBV, U22 FAN3214, U23 FAN3214, U24 CSD17506Q5A, U25 CSD17506Q5A, U27 CSD17506Q5A, U3 SN74LVC1G08DBV, U30 ISO7221, U31 ISO7221, U32 PDS1-S5-S5-M-TR, U33 ISO7221, U34 ISO7221, U35 PDS1-S5-S5-M-TR, U36 ADC121S021, U37 ADC121S021, U38 FT232RL, U42 TPS54540DDARQ1, U5 CD4050BD, U6 CD4050BD, U7 MCP2562FD, U8 ADUM3160BRWZ-RL, Y2 16MHz

Commit message: ez
Parts:
- removed JP5: (no value), adafruit:1X06-CLEANBIG
- removed SV1, SV2: (no value), con-lstb:MA04-1
- added J4, J6: MOLEX_43650-0416MOLEX_43650-0416_0_0, FormE:MOLEX_43650-0416_0
- added J7: 43650-0616, FormE:MOLEX_43650-0616
- moved Q1 169.7 mm to (21.6, 64.1), turned to 180 degrees
- moved R2 152.7 mm to (15.9, 29.8), turned to 270 degrees
- moved C51 118.1 mm to (-132.1, 227.3)
- moved C53 118.1 mm to (-132.1, 222.2)
- moved R57 118.1 mm to (-132.1, 201.9)
- moved C1 118.1 mm to (-152.4, 212.1)
- moved C21 118.1 mm to (-132.1, 217.2)
- moved C4 118.1 mm to (-162.6, 212.1)
- moved C43 118.1 mm to (-106.7, 222.2)
- moved C46 118.1 mm to (-111.8, 222.2)
- moved C52 118.1 mm to (-166.4, 227.3)
- moved C56 118.1 mm to (-142.2, 222.2)
- moved C65 118.1 mm to (-152.4, 222.2)
- moved C7 118.1 mm to (-177.8, 212.1)
- moved C70 118.1 mm to (-142.2, 227.3)
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Connections:
- removed net BATTERY_VOLTAGE_MONITOR_MISO: U33.P$6, U4.31
- removed net BATTERY_VOLTAGE_MONITOR_SCLK: U34.P$7, U4.25
- removed net VEHICLE_VOLTAGE_MISO: U30.P$6, U4.94
- removed net VEHICLE_VOLTAGE_MONITOR_SCLK: U31.P$7, U4.95
- new net VOLTAGE_MONITOR_MISO: U30.P$6, U33.P$6, U4.94
- new net VOLTAGE_MONITOR_SCLK: U31.P$7, U34.P$7, U4.95
- net +5V/1: now also J7.4; no longer JP5.4
- net BATTERY_VOLTAGE_MONITOR_CS: no longer U4.24
- net BMS_FAULT_HV: now also J7.5; no longer JP5.5
- net BMS_RX_HV: now also J7.2; no longer JP5.2
- net BMS_TX_HV: now also J7.3; no longer JP5.3
- net GND1: now also J7.6; no longer JP5.6
- net GND2: now also J4.3, J4.4; no longer SV1.1, SV1.2
- net GND3: now also J6.3, J6.4; no longer SV2.1, SV2.2
- net N$102: now also J4.1, J4.2; no longer SV1.3, SV1.4
- net N$111: now also J6.2; no longer SV2.3
- net N$112: now also J6.1; no longer SV2.4
- net WAKEUP_HV: now also J7.1; no longer JP5.1
Routing:
- net POS_GATE: track 0.00 -> 8.76 mm
- net NEG_GATE: track 0.00 -> 8.12 mm
- net IMD_GND: track 0.00 -> 7.93 mm
- net CAR_CAN_P: track 0.00 -> 5.81 mm
- net CAR_CAN_N: track 0.00 -> 5.75 mm
- net PRECH_GATE: track 0.00 -> 3.42 mm
- net GND: track 0.00 -> 3.23 mm, vias 0 -> 12
- net +15V: track 0.00 -> 2.02 mm, vias 0 -> 2
- added copper zone on layer 15, net +15V
- added copper zone on layer 1, net GND
- added copper zone on layer 1, net N$30
- added copper zone on layer 1, net N$97
- added copper zone on layer 1, net NEG_FET
- added copper zone on layer 1, net POS_FET
- added copper zone on layer 1, net PRE_FET
- added copper zone on layer 1, net SHUTDOWN_CIRCUIT_FROM_OUTSIDE

Commit message: HV isolation, 5V supply
Parts:
- added U$1: (no value), FormE:BENDER-ISOMETER
- moved C93 391.3 mm to (169.5, 20.3), turned to 270 degrees
- moved R96 383.7 mm to (173.4, 21.6), turned to 180 degrees
- moved R26 369.3 mm to (132.7, 27.9)
- moved U34 360.5 mm to (150.5, 38.1)
- moved R97 356.9 mm to (138.4, 23.5), turned to 90 degrees
- moved C3 356.9 mm to (135.9, 24.1), turned to 180 degrees
- moved C5 353.9 mm to (136.5, 31.1), turned to 180 degrees
- moved U33 348.8 mm to (145.4, 38.1)
- moved C92 318.4 mm to (141.6, 27.9)
- moved C90 316.8 mm to (151.1, 29.8), turned to 270 degrees
- moved C89 307.4 mm to (144.1, 29.8), turned to 270 degrees
- moved D7 294.0 mm to (42.5, 74.9), turned to 180 degrees
- moved C94 272.3 mm to (48.3, 64.8), turned to 270 degrees
- moved C99 265.6 mm to (52.1, 57.8), turned to 180 degrees
- moved R51 247.5 mm to (41.3, 62.2), turned to 90 degrees
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Routing:
- net +5V/3: track 0.00 -> 43.4 mm, vias 0 -> 3
- net GND3: track 0.00 -> 22.7 mm, vias 0 -> 11
- net N$94: track 0.00 -> 14.0 mm
- net N$104: track 0.00 -> 11.6 mm
- net N$105: track 0.00 -> 10.8 mm
- net 5VREG_EN1: track 0.00 -> 8.39 mm
- net N$96: track 0.00 -> 6.11 mm
- net BATTERY_VOLTAGE_FB: track 0.00 -> 5.12 mm
- net COMP_5V2: track 0.00 -> 4.80 mm
- net USB_D_N: track 0.00 -> 4.77 mm, vias 0 -> 1
- net USB_D_P: track 0.00 -> 4.51 mm, vias 0 -> 1
- net VEHICLE_VOLTAGE_FB: track 0.00 -> 4.50 mm
- net FB_5V2: track 0.00 -> 4.30 mm
- net GND: track 3.23 -> 7.15 mm, vias 12 -> 39
- net N$114: track 0.00 -> 3.68 mm
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- added copper zone on layer 1, net +15V
- added copper zone on layer 1, net +5V
- added copper zone on layer 1, net GND3
- added copper zone on layer 16, net GND3
- added copper zone on layer 1, net N$100
- added copper zone on layer 1, net N$101
- added copper zone on layer 1, net N$102
- added copper zone on layer 1, net N$110
- added copper zone on layer 1, net N$111
- added copper zone on layer 1, net N$112
- added copper zone on layer 1, net N$114
- added copper zone on layer 1, net N$117
- added copper zone on layer 1, net SW_5V2

Commit message: rough
Parts:
- added C28: 4.7uF, rcl:C0603K
- moved C81 429.6 mm to (196.8, 41.9), turned to 180 degrees
- moved R27 427.6 mm to (196.8, 38.1), turned to 180 degrees
- moved C87 416.6 mm to (176.5, 40.0), turned to 270 degrees
- moved JP4 362.8 mm to (119.4, 8.26), turned to 270 degrees
- moved U31 362.3 mm to (183.5, 48.9)
- moved U30 360.7 mm to (177.8, 48.9)
- moved JP6 360.1 mm to (122.6, 30.5)
- moved JP3 353.6 mm to (114.9, 8.26), turned to 270 degrees
- moved JP2 352.2 mm to (121.3, 10.8), turned to 90 degrees
- moved R1 349.4 mm to (110.5, 9.53), turned to 90 degrees
- moved C91 345.1 mm to (181.0, 29.2)
- moved JP1 343.5 mm to (116.8, 10.2), turned to 90 degrees
- moved C88 327.3 mm to (182.9, 41.3)
- moved U11 315.2 mm to (123.2, 22.2)
- moved C20 314.7 mm to (106.7, 6.35), turned to 180 degrees
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Connections:
- net BMS_CAN_N renamed HV_BMS_CAN_N
- net BMS_CAN_P renamed HV_BMS_CAN_P
- new net HV_BMS_CAN_RX: JP1.3, U13.4
- new net HV_BMS_CAN_TX: JP2.3, U13.1
- net +5V/1: now also C28.1
- net BMS_CAN_RX: no longer JP1.3, U13.4
- net BMS_CAN_TX: no longer JP2.3, U13.1
- net BMS_FAULT: now also U11.P$6; no longer U10.P$6
- net BMS_FAULT_HV: now also U11.P$3; no longer U10.P$3
- net BMS_RX: now also U10.P$6; no longer U11.P$6
- net GND1: now also C28.2
- net N$31: now also U10.P$3; no longer U11.P$3
Routing:
- net +5V/2: track 0.00 -> 73.5 mm, vias 0 -> 5
- net GND: track 7.15 -> 37.6 mm, vias 39 -> 46
- net FAULT_IMD_PRE-BUFFER: track 0.00 -> 28.4 mm
- net M_LS: track 0.00 -> 27.0 mm
- net +15V: track 5.28 -> 30.0 mm, vias 4 -> 6
- net +5V/1: track 0.00 -> 24.0 mm, vias 0 -> 8
- net WAKEUP_HV: track 0.00 -> 21.1 mm
- net GND2: track 1.06 -> 21.5 mm, vias 1 -> 11
- net HV_BMS_CAN_TX: track 0.00 -> 20.1 mm, vias 0 -> 2
- net BMS_FAULT_HV: track 0.00 -> 18.8 mm
- net HV_BMS_CAN_RX: track 0.00 -> 16.9 mm, vias 0 -> 2
- net GND1: track 0.00 -> 15.7 mm, vias 0 -> 9
- net HV_BMS_CAN_P: track 0.00 -> 15.6 mm, vias 0 -> 2
- net N$93: track 0.00 -> 14.4 mm
- net N$92: track 0.00 -> 14.0 mm
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- added copper zone on layer 15, net +5V/1
- added copper zone on layer 1, net +5V/2
- added copper zone on layer 1, net +5V/3
- added copper zone on layer 1, net GND1
- added copper zone on layer 16, net GND1
- added copper zone on layer 1, net GND2
- added copper zone on layer 16, net GND2
- added copper zone on layer 1, net N$6
Other:
- board text added: "+"
- board text added: "-"
- board text added: "BATTERY (INSIDE)"
- board text added: "VEHICLE (OUTSIDE)"

Commit message: routing
Parts:
- removed S3: TE-FSM4JSMATR, FormE:TE-FSM4JSMATR
- added S2: 147873-2, FormE:TE-147873-2
- moved C35 235.0 mm to (102.2, 84.5), turned to 45 degrees
- moved C34 235.0 mm to (107.3, 80.0), turned to 45 degrees
- moved C33 230.6 mm to (107.3, 60.3), turned to 315 degrees
- moved C32 229.6 mm to (111.8, 64.8), turned to 315 degrees
- moved C37 228.6 mm to (85.7, 82.5), turned to 135 degrees
- moved C36 227.1 mm to (88.3, 55.9), turned to 225 degrees
- moved C31 222.2 mm to (109.2, 62.2), turned to 315 degrees
- moved C1 211.6 mm to (113.0, 66.0), turned to 315 degrees
- moved C2 203.6 mm to (101.0, 85.7), turned to 45 degrees
- moved C48 201.8 mm to (87.0, 83.8), turned to 135 degrees
- moved C55 189.3 mm to (105.1, 58.7), turned to 315 degrees
- moved C53 181.7 mm to (102.9, 56.5), turned to 315 degrees
- moved C49 177.7 mm to (104.1, 57.8), turned to 315 degrees
- moved C51 164.0 mm to (84.5, 58.4), turned to 45 degrees
- moved C54 162.0 mm to (80.0, 80.0), turned to 135 degrees
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Connections:
- net GND: now also S2.P$2; no longer S3.3, S3.4
- net N$63: now also S2.P$1; no longer S3.1, S3.2
Routing:
- net +5V: track 6.50 -> 192.0 mm, vias 1 -> 12
- net PRECHARGE_CONTACTOR_CTRL: track 0.00 -> 138.0 mm, vias 0 -> 6
- net CAR_CAN_TX: track 0.00 -> 128.7 mm, vias 0 -> 4
- net CAR_CAN_RX: track 0.00 -> 125.5 mm, vias 0 -> 6
- net NEGATIVE_CONTACTOR_CTRL: track 0.00 -> 121.1 mm, vias 0 -> 3
- net CONTACTOR_OPEN_3V3: track 0.00 -> 115.4 mm, vias 0 -> 5
- net POSITIVE_CONTACTOR_CTRL: track 0.00 -> 111.7 mm, vias 0 -> 3
- net CONTACTOR_CLOSED_3V3: track 0.00 -> 101.7 mm, vias 0 -> 4
- net FAULT_AMS_INDICATOR: track 0.00 -> 98.5 mm, vias 0 -> 6
- net BMS_FAULT: track 0.00 -> 95.2 mm, vias 0 -> 3
- net WAKEUP: track 4.55 -> 89.6 mm, vias 0 -> 3
- net +3V3: track 8.60 -> 93.0 mm, vias 2 -> 33
- net GND: track 37.6 -> 116.4 mm, vias 46 -> 98
- net 5KW_3V3: track 0.00 -> 74.0 mm, vias 0 -> 4
- net N$11: track 0.00 -> 73.7 mm, vias 0 -> 4
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- added copper zone on layer 15, net +1V2
- added copper zone on layer 15, net +3V3
- added copper zone on layer 15, net +5V
Other:
- board text added: "3v3"
- board text added: "5V"
- board text added: "RX"
- board text added: "TX"

Commit message: Continued layout
Parts:
- moved C70 11.1 mm to (49.5, 88.9), turned to 270 degrees
- moved L6 10.2 mm to (57.8, 80.6), turned to 270 degrees
- moved C72 9.69 mm to (59.7, 78.7), turned to 270 degrees
- moved L5 9.03 mm to (47.0, 92.1)
- moved C40 7.85 mm to (47.0, 84.5)
- moved U18 7.65 mm to (54.0, 80.6), turned to 270 degrees
- moved U16 5.85 mm to (47.0, 88.3)
- moved C71 3.24 mm to (50.8, 82.5), turned to 90 degrees
Connections:
- net 5KW_3V3: now also U14.2
- net CURRENT_SENSE_-750_TO_750A: now also H3.4; no longer H3.5
- net CURRENT_SENSE_-75_TO_75A: now also H3.5; no longer H3.4
- net INDICATOR_2: no longer U4.127
- net INDICATOR_3: no longer U14.2
Routing:
- net +5V: track 192.0 -> 53.7 mm, vias 12 -> 15
- net BATTERY_VOLTAGE_MONITOR_CS: track 0.00 -> 99.3 mm, vias 0 -> 2
- net BMS_CAN_TX: track 0.00 -> 84.9 mm, vias 0 -> 2
- net BMS_CAN_RX: track 0.00 -> 76.6 mm, vias 0 -> 3
- net 5KW_3V3: track 74.0 -> 120.8 mm, vias 4 -> 5
- net UART_RX: track 8.94 -> 55.5 mm, vias 0 -> 1
- net UART_TX: track 8.15 -> 53.4 mm, vias 0 -> 1
- net BMS_UART_TX: track 0.00 -> 44.3 mm, vias 0 -> 2
- net BMS_UART_RX: track 0.00 -> 39.9 mm, vias 0 -> 2
- net +3V3: track 93.0 -> 100.7 mm, vias 33 -> 35
- net GND: track 116.4 -> 123.6 mm, vias 98 -> 104
- net BATTERY_VOLTAGE_IS_AVAILABLE: track 0.00 -> 6.89 mm
- net INDICATOR_2: track 21.4 -> 15.4 mm
- net N$57: track 0.00 -> 2.26 mm
- net N$59: track 0.00 -> 2.26 mm
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- added copper zone on layer 1, net +1V2
- added copper zone on layer 2, net +5V
